File: eagle/s0httpv8.brd (EAGLE design)
At the start: 33 parts, among them X1 MKDSN1,5/6-5,08, X2 MKDSN1,5/6-5,08

Commit message: added v8, added stiker, updated pinning in sketch
Parts:
- removed R23, R24: (no value), resistor:R0805
- added JP3: (no value), jumper:JP2
- JP2: device jumper:JP7Q -> jumper:JP2
- moved U$13 5.15 mm to (46.2, 5.00), turned to 90 degrees
- moved U$9 4.20 mm to (70.2, 8.70), turned to 270 degrees
- moved U$10 3.96 mm to (70.2, 12.4), turned to 270 degrees
- moved U$11 3.71 mm to (70.2, 16.2), turned to 270 degrees
- moved JP2 2.76 mm to (29.8, 5.75), turned to 180 degrees
- moved R4 2.76 mm to (44.5, 22.0)
- moved U$1 2.76 mm to (51.3, 26.0)
- moved R2 2.51 mm to (44.5, 20.0)
- moved U$12 2.46 mm to (70.2, 19.9), turned to 270 degrees
- moved R11 1.68 mm to (8.00, 4.75), turned to 0 degrees
- moved U$7 1.26 mm to (12.0, 9.80), turned to 90 degrees
- moved U$5 1.06 mm to (12.0, 18.1), turned to 90 degrees
- moved U$6 1.06 mm to (12.0, 13.8), turned to 90 degrees
- moved U$8 1.06 mm to (12.0, 5.55), turned to 90 degrees
- moved U$4 0.89 mm to (12.0, 22.1), turned to 90 degrees
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Connections:
- removed net N$20: JP2.10, R24.1
- removed net N$31: JP2.1, JP2.11, JP2.13, JP2.3, JP2.5, JP2.7, JP2.9, U$1.GND2, U$2.GNDOUT, U$3.S, U$4.S, U$5.S, U$6.S, U$7.S, U$8.S
- removed net N$32: JP1.1, JP1.2, JP1.3, U$1.GND1
- removed net N$36: JP2.12, R23.1
- removed net N$38: R23.2, U$1.A3
- removed net N$39: R24.2, U$1.A2
- removed net VDD: U$10.S, U$11.S, U$12.S, U$2.GNDIN, U$9.S, X2.5
- new net GND: JP1.1, JP1.2, JP1.3, JP2.2, U$1.GND1, U$1.GND2, U$10.S, U$11.S, U$12.S, U$2.GNDIN, U$2.GNDOUT, U$3.S, U$4.S, U$5.S, U$6.S, U$7.S, U$8.S, U$9.S, X2.5
- net N$12: now also JP2.1
- net N$13: now also U$1.A3; no longer U$1.A5
- net N$16: now also U$1.A2; no longer U$1.A4
- net N$3: now also JP3.3; no longer JP2.2
- net N$6: now also JP3.2; no longer JP2.4
- net N$7: now also JP3.1; no longer JP2.6
- net N$9: now also JP2.3; no longer JP2.8
Routing:
- net N$31: track 84.4 -> 0.00 mm
- net VDD: track 40.3 -> 0.00 mm
- net N$12: track 13.4 -> 31.4 mm
- net N$32: track 18.0 -> 0.00 mm
- net N$19: track 7.35 -> 17.6 mm
- net N$13: track 35.5 -> 43.7 mm
- net N$16: track 37.0 -> 43.3 mm
- net VCC: track 216.6 -> 220.9 mm
- net N$39: track 3.96 -> 0.00 mm
- net N$21: track 44.1 -> 47.7 mm
- net N$36: track 3.40 -> 0.00 mm
- net N$33: track 16.5 -> 19.7 mm
- net N$38: track 3.21 -> 0.00 mm
- net N$1: track 12.0 -> 14.8 mm
- net N$20: track 2.48 -> 0.00 mm
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- added copper zone on layer 16, net GND
Other:
- board text added: "s0http v8"
- board text removed: "s0http_v6"
